Commit message: WIP Etapa 3: cobertura autonoma (LiDAR detecta proprio chassi, pendente fix)

File: src/mower_description/urdf/mower.urdf.xacro (robot description, xacro)
@@ -142,5 +142,5 @@
     <child link="lidar_link"/>
     <!-- LiDAR montado no centro do chassi, 5cm acima do topo -->
-    <origin xyz="0 0 ${chassis_height + 0.05}" rpy="0 0 0"/>
+    <origin xyz="0 0 ${chassis_height + 0.10}" rpy="0 0 0"/>
   </joint>
   <!-- ============ PLUGINS GAZEBO ============ -->
